Commit message: Upload some notebooks for inverse kin and dumb control

File: models/SimpleWalker/urdf/SimpleWalker.urdf (robot description, URDF)
Before this commit: robot SimpleWalker, 28 links, 27 joints
Links:
- removed link Link_0
- added link BaseLink, mass 1.0; collision box size=1.2 1.0 0.5; visual box size=1.2 1.0 0.5
Joints:
- removed joint Gripper1
- removed joint Gripper2
- removed joint GripperBase
- added joint Gripper_LeftGrip: type prismatic, parent GripperBase, child Gripper2, origin xyz=0.53 0 -0.05 rpy=3.14159 0 0, axis 0 0 1.0, limit lower=0 upper=0.4 effort=500.0 velocity=20.0
- added joint Gripper_Revolute: type revolute, parent BaseLink, child GripperBase, origin xyz=0.6 0 0 rpy=1.5708 0 0, axis 0 0 1.0, limit lower=-3.0 upper=3.0 effort=500.0 velocity=20.0
- added joint Gripper_RightGrip: type prismatic, parent GripperBase, child Gripper1, origin xyz=0.53 0 0.05 rpy=0 0 0, axis 0 0 1.0, limit lower=0 upper=0.4 effort=500.0 velocity=20.0
- joint Joint_1: parent Link_0 -> BaseLink
- joint Joint_13: parent Link_0 -> BaseLink
- joint Joint_17: parent Link_0 -> BaseLink
- joint Joint_21: parent Link_0 -> BaseLink
- joint Joint_5: parent Link_0 -> BaseLink
- joint Joint_9: parent Link_0 -> BaseLink
